File: hx4k_dev_board/hx4k_dev_board.kicad_pcb (KiCad board)
At the start: 4 copper layers, 85 x 54 mm, 117 parts, among them J1 USB_B, J2 RB1-125B8G1A, J3 Conn_01x08, J4 Conn_02x06_Odd_Even, J5 Conn_02x06_Odd_Even, SW1 SW_SPST, SW2 SW_SPST, SW3 SW_SPST, U1 W9812G6KH-6, U2 CH340E, U3 TPS7A7001DDA, U4 TPS7A7001DDA, U5 RTL8211EG-VB-CG, U6 ICE40HX4K-TQ144, U7 W25Q128JVS, X1 SG-7050CAN, X2 SG-7050CAN

Commit message: Add EEPROM
Parts:
- added C38: 100n, Capacitor_SMD:C_0603_1608Metric, F.Cu at (171.8, 89.7)
- added R40: 10k, Resistor_SMD:R_0603_1608Metric, F.Cu at (168.7, 96.6)
- added R41: 10k, Resistor_SMD:R_0603_1608Metric, F.Cu at (167.2, 96.6)
- added U8: M24C01-RMN, Package_SO:SOIC-8_3.9x4.9mm_P1.27mm, F.Cu at (167.4, 92.4)
- moved C13 180.9 mm to (137.9, 111.7)
- moved C20 180.9 mm to (164.4, 109.1)
- moved C35 180.9 mm to (155.6, 99.4)
- moved D1 180.9 mm to (143.9, 83.4)
- moved R13 180.9 mm to (155.7, 112.5)
- moved R14 180.9 mm to (156.9, 100.7)
- moved R15 180.9 mm to (156.3, 110.9)
- moved R16 180.9 mm to (157.1, 109.4)
- moved R21 180.9 mm to (116.6, 97.0)
- moved R25 180.9 mm to (161.4, 93.6)
- moved R9 180.9 mm to (142.4, 107.2)
- moved C1 180.9 mm to (196.8, 105.0)
- moved C10 180.9 mm to (131.8, 89.0)
- moved C11 180.9 mm to (141.3, 87.8)
- moved C12 180.9 mm to (141.3, 94.3)
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Connections:
- U6 pad 134: Net-(U6-Pad134) -> /EEPROM/SCL
- U6 pad 135: Net-(U6-Pad135) -> /EEPROM/SDA
Routing:
- net /EEPROM/SDA: track 0.00 -> 21.6 mm, vias 0 -> 1
- net /EEPROM/SCL: track 0.00 -> 20.4 mm, vias 0 -> 1
- net GND: track 82.1 -> 88.4 mm, vias 76 -> 79
- net +3V3: track 72.3 -> 77.3 mm, vias 50 -> 52
Other:
- board text added: "TODO: Change Via size to JLC standard"

Commit message: Tidy up
Parts:
- moved R1 1.25 mm to (127.4, 77.5)
Routing:
- net Net-(J1-Pad5): track 15.0 -> 16.6 mm
Other:
- net class 100R diff: via_dia 0.53 -> 0.45
- net class 50R: via_dia 0.53 -> 0.45
- net class 90R: via_dia 0.53 -> 0.45
- net class Default: via_dia 0.53 -> 0.45
- net class Power: via_dia 0.53 -> 0.45
- rule via_min_size: 0.53 -> 0.45
- board text added: "Controlled impedance designed for JLC2313 stackup"
- board text added: "Designed by Joshua Tyler October 2019"
- board text added: "Designed to JLCPCB Design rules"
- board text added: "KiCAD doesn't suport separate track to track and via to track clearence. To combat this, the board was designed with 0.53mm vias, later shrunk to 0.45mm after final design rule check."
- board text removed: "JLC2313 stackup"
