File: hw/POWER.sch (KiCad schematic (older format))
At the start: 10 parts, among them U3 TPS7A7001DDA, U4 TPS7A7001DDA

Commit message: Add comment
Other:
- note added: "iCE40 has no particular requirements on power sequencing.\n\n2A on each rail will be plenty."
Changed lines of the file:
@@
 Connection ~ 6250 2300
 Connection ~ 3450 2300
+Text Notes 7750 1550 0    50   ~ 0
+iCE40 has no particular requirements on power sequencing.\n\n2A on each rail will be plenty.
 $EndSCHEMATC
