File: hw/manila_ice.kicad_pcb (KiCad board)
At the start: 4 copper layers, 85 x 54 mm, 122 parts, among them J1 USB_B, J2 RB1-125B8G1A, J3 Conn_01x08, J4 Conn_02x06_Odd_Even, J5 Conn_02x06_Odd_Even, SW1 SW_SPST, SW2 SW_SPST, SW3 SW_SPST, U1 W9812G6KH-6, U2 CH340E, U3 TPS7A7001DDA, U4 TPS7A7001DDA, U5 RTL8211EG-VB-CG, U6 ICE40HX4K-TQ144, U7 W25Q128JVS, U8 M24C01-RMN, X1 SG-7050CAN, X2 SG-7050CAN

Commit message: Finished except some parts need to be rotated
Routing:
- net /ETHERNET/MDI3_N: track 16.0 -> 35.1 mm
- net /ETHERNET/MDI3_P: track 17.4 -> 33.5 mm
- net /ETHERNET/MDI1_P: track 18.1 -> 28.4 mm, vias 1 -> 2
- net /ETHERNET/MDI1_N: track 16.4 -> 25.7 mm, vias 1 -> 2
- net /ETHERNET/VDD: track 0.00 -> 5.72 mm, vias 0 -> 9
- net /ETHERNET/MDI0_N: track 16.6 -> 17.3 mm
- net /ETHERNET/MDI0_P: track 18.8 -> 19.5 mm
- net /ETHERNET/CLK50: track 13.7 -> 14.3 mm
- added copper zone on B.Cu, net /ETHERNET/VDD
Other:
- rule solder_mask_min_width: 0.25 -> 0.0889
- board text removed: "TODO: Change Via size to JLC standard"
