File: hw/LEDS.sch (KiCad schematic (older format))
At the start: 16 parts

Commit message: Fix JLC rotation
Parts:
- D10, D11, D4, D5, D6, D7, D8, D9, R32, R33, R34, R35, R36, R37, R38, R39: JLCPCB Rotation (none) -> 0
