File: hw/USB_UART.sch (KiCad schematic (older format))
At the start: 4 parts, among them U2 CH340E

Commit message: Add ability to rotate part for JLC PCB
Parts:
- U2: JLCPCB Rotation (none) -> -90
Changed lines of the file:
@@
 F 3 "https://www.mpja.com/download/35227cpdata.pdf" H 5300 4850 50  0001 C CNN
 F 4 "C99652" H 5400 4700 50  0001 C CNN "LCSC Part"
+F 5 "-90" H 5650 4050 50  0001 C CNN "JLCPCB Rotation"
 	1    5650 4050
 	1    0    0    -1

Commit message: Fix JLC rotation
Parts:
- C8, D1, R2: JLCPCB Rotation (none) -> 0
Changed lines of the file:
@@
 U 1 1 5D7CE99F
 P 5650 4050
-F 0 "U2" H 5400 4600 50  0000 C CNN
-F 1 "CH340E" H 5900 4600 50  0000 C CNN
-F 2 "Package_SO:MSOP-10_3x3mm_P0.5mm" H 5700 3500 50  0001 L CNN
-F 3 "https://www.mpja.com/download/35227cpdata.pdf" H 5300 4850 50  0001 C CNN
-F 4 "-90" H 5650 4050 50  0001 C CNN "JLCPCB Rotation"
-F 5 "C99652" H 5400 4700 50  0001 C CNN "LCSC Part"
+F 0 "U2" H 5400 4600 50 0000 C CNN
+F 1 "CH340E" H 5900 4600 50 0000 C CNN
+F 2 "Package_SO:MSOP-10_3x3mm_P0.5mm" H 5700 3500 50 0001 L CNN
+F 3 "https://www.mpja.com/download/35227cpdata.pdf" H 5300 4850 50 0001 C CNN
+F 4 "-90" H 5650 4050 50 0001 C CNN "JLCPCB Rotation"
+F 5 "C99652" H 5400 4700 50 0001 C CNN "LCSC Part"
 	1    5650 4050
 	1    0    0    -1
@@
 U 1 1 5D7D3316
 P 5650 4700
-F 0 "#PWR021" H 5650 4450 50  0001 C CNN
-F 1 "GND" H 5655 4527 50  0000 C CNN
-F 2 "" H 5650 4700 50  0001 C CNN
-F 3 "" H 5650 4700 50  0001 C CNN
+F 0 "#PWR021" H 5650 4450 50 0001 C CNN
+F 1 "GND" H 5655 4527 50 0000 C CNN
+F 2 "" H 5650 4700 50 0001 C CNN
+F 3 "" H 5650 4700 50 0001 C CNN
 	1    5650 4700
 	1    0    0    -1
@@
 U 1 1 5D7D0D58
 P 6850 4450
-F 0 "R2" H 6920 4496 50  0000 L CNN
-F 1 "1k" H 6920 4405 50  0000 L CNN
-F 2 "Resistor_SMD:R_0603_1608Metric" V 6780 4450 50  0001 C CNN
-F 3 "~" H 6850 4450 50  0001 C CNN
-F 4 "C21190" H 6920 4596 50  0001 C CNN "LCSC Part"
+F 0 "R2" H 6920 4496 50 0000 L CNN
+F 1 "1k" H 6920 4405 50 0000 L CNN
+F 2 "Resistor_SMD:R_0603_1608Metric" V 6780 4450 50 0001 C CNN
+F 3 "~" H 6850 4450 50 0001 C CNN
+F 4 "0" H 6920 4596 50 0001 C CNN "JLCPCB Rotation"
+F 5 "C21190" H 6920 4596 50 0001 C CNN "LCSC Part"
 	1    6850 4450
 	1    0    0    -1
@@
 U 1 1 5D7CFA7C
 P 6850 4800
-F 0 "D1" V 6889 4683 50  0000 R CNN
-F 1 "LED" V 6798 4683 50  0000 R CNN
-F 2 "Diode_SMD:D_0805_2012Metric_Castellated" H 6850 4800 50  0001 C CNN
-F 3 "~" H 6850 4800 50  0001 C CNN
-F 4 "C84256" H 6889 4783 50  0001 C CNN "LCSC Part"
+F 0 "D1" V 6889 4683 50 0000 R CNN
+F 1 "LED" V 6798 4683 50 0000 R CNN
+F 2 "Diode_SMD:D_0805_2012Metric_Castellated" H 6850 4800 50 0001 C CNN
+F 3 "~" H 6850 4800 50 0001 C CNN
+F 4 "0" H 6889 4783 50 0001 C CNN "JLCPCB Rotation"
+F 5 "C84256" H 6889 4783 50 0001 C CNN "LCSC Part"
 	1    6850 4800
 	0    -1   -1   0
@@
 U 1 1 5D7D83DF
 P 6850 5000
-F 0 "#PWR022" H 6850 4750 50  0001 C CNN
-F 1 "GND" H 6855 4827 50  0000 C CNN
-F 2 "" H 6850 5000 50  0001 C CNN
-F 3 "" H 6850 5000 50  0001 C CNN
+F 0 "#PWR022" H 6850 4750 50 0001 C CNN
+F 1 "GND" H 6855 4827 50 0000 C CNN
+F 2 "" H 6850 5000 50 0001 C CNN
+F 3 "" H 6850 5000 50 0001 C CNN
 	1    6850 5000
 	1    0    0    -1
@@
 U 1 1 5D7DBD9C
 P 5650 3350
-F 0 "#PWR020" H 5650 3200 50  0001 C CNN
-F 1 "+3V3" H 5665 3523 50  0000 C CNN
-F 2 "" H 5650 3350 50  0001 C CNN
-F 3 "" H 5650 3350 50  0001 C CNN
+F 0 "#PWR020" H 5650 3200 50 0001 C CNN
+F 1 "+3V3" H 5665 3523 50 0000 C CNN
+F 2 "" H 5650 3350 50 0001 C CNN
+F 3 "" H 5650 3350 50 0001 C CNN
 	1    5650 3350
 	1    0    0    -1
@@
 U 1 1 5D7DCA49
 P 4400 3150
-F 0 "C8" H 4515 3196 50  0000 L CNN
-F 1 "100n" H 4515 3105 50  0000 L CNN
-F 2 "Capacitor_SMD:C_0603_1608Metric" H 4438 3000 50  0001 C CNN
-F 3 "~" H 4400 3150 50  0001 C CNN
-F 4 "C14663" H 4515 3296 50  0001 C CNN "LCSC Part"
+F 0 "C8" H 4515 3196 50 0000 L CNN
+F 1 "100n" H 4515 3105 50 0000 L CNN
+F 2 "Capacitor_SMD:C_0603_1608Metric" H 4438 3000 50 0001 C CNN
+F 3 "~" H 4400 3150 50 0001 C CNN
+F 4 "0" H 4515 3296 50 0001 C CNN "JLCPCB Rotation"
+F 5 "C14663" H 4515 3296 50 0001 C CNN "LCSC Part"
 	1    4400 3150
 	1    0    0    -1
@@
 U 1 1 5D7DCD2D
 P 4400 2950
-F 0 "#PWR018" H 4400 2800 50  0001 C CNN
-F 1 "+3V3" H 4415 3123 50  0000 C CNN
-F 2 "" H 4400 2950 50  0001 C CNN
-F 3 "" H 4400 2950 50  0001 C CNN
+F 0 "#PWR018" H 4400 2800 50 0001 C CNN
+F 1 "+3V3" H 4415 3123 50 0000 C CNN
+F 2 "" H 4400 2950 50 0001 C CNN
+F 3 "" H 4400 2950 50 0001 C CNN
 	1    4400 2950
 	1    0    0    -1
@@
 U 1 1 5D7DD32D
 P 4400 3350
-F 0 "#PWR019" H 4400 3100 50  0001 C CNN
-F 1 "GND" H 4405 3177 50  0000 C CNN
-F 2 "" H 4400 3350 50  0001 C CNN
-F 3 "" H 4400 3350 50  0001 C CNN
+F 0 "#PWR019" H 4400 3100 50 0001 C CNN
+F 1 "GND" H 4405 3177 50 0000 C CNN
+F 2 "" H 4400 3350 50 0001 C CNN
+F 3 "" H 4400 3350 50 0001 C CNN
 	1    4400 3350
 	1    0    0    -1
