File: hw/EEPROM.sch (KiCad schematic (older format))
At the start: 2 parts, among them U8 M24C01-RMN

Commit message: Add outputs folder
Parts:
- U8: LCSC Part (none) -> C79988
Changed lines of the file:
@@
 EESchema Schematic File Version 4
-LIBS:hx4k_dev_board-cache
 EELAYER 30 0
 EELAYER END
@@
 F 2 "Package_SO:SOIC-8_3.9x4.9mm_P1.27mm" H 5600 3750 50  0001 C CNN
 F 3 "http://www.st.com/content/ccc/resource/technical/document/datasheet/b0/d8/50/40/5a/85/49/6f/DM00071904.pdf/files/DM00071904.pdf/jcr:content/translations/en.DM00071904.pdf" H 5650 2900 50  0001 C CNN
+F 4 "C79988" H 5600 3400 50  0001 C CNN "LCSC Part"
 	1    5600 3400
 	1    0    0    -1

Commit message: Fix JLC rotation
Parts:
- C38: JLCPCB Rotation (none) -> 0
- U8: JLCPCB Rotation (none) -> -90
Changed lines of the file:
@@
 U 1 1 5DAA4F4F
 P 5600 3400
-F 0 "U8" H 5350 3650 50  0000 C CNN
-F 1 "M24C01-RMN" H 5950 3650 50  0000 C CNN
-F 2 "Package_SO:SOIC-8_3.9x4.9mm_P1.27mm" H 5600 3750 50  0001 C CNN
-F 3 "http://www.st.com/content/ccc/resource/technical/document/datasheet/b0/d8/50/40/5a/85/49/6f/DM00071904.pdf/files/DM00071904.pdf/jcr:content/translations/en.DM00071904.pdf" H 5650 2900 50  0001 C CNN
-F 4 "C79988" H 5600 3400 50  0001 C CNN "LCSC Part"
+F 0 "U8" H 5350 3650 50 0000 C CNN
+F 1 "M24C01-RMN" H 5950 3650 50 0000 C CNN
+F 2 "Package_SO:SOIC-8_3.9x4.9mm_P1.27mm" H 5600 3750 50 0001 C CNN
+F 3 "http://www.st.com/content/ccc/resource/technical/document/datasheet/b0/d8/50/40/5a/85/49/6f/DM00071904.pdf/files/DM00071904.pdf/jcr:content/translations/en.DM00071904.pdf" H 5650 2900 50 0001 C CNN
+F 4 "-90" H 5350 3750 50 0001 C CNN "JLCPCB Rotation"
+F 5 "C79988" H 5600 3400 50 0001 C CNN "LCSC Part"
 	1    5600 3400
 	1    0    0    -1
@@
 U 1 1 5DAA54F8
 P 5150 3800
-F 0 "#PWR0130" H 5150 3550 50  0001 C CNN
-F 1 "GND" H 5155 3627 50  0000 C CNN
-F 2 "" H 5150 3800 50  0001 C CNN
-F 3 "" H 5150 3800 50  0001 C CNN
+F 0 "#PWR0130" H 5150 3550 50 0001 C CNN
+F 1 "GND" H 5155 3627 50 0000 C CNN
+F 2 "" H 5150 3800 50 0001 C CNN
+F 3 "" H 5150 3800 50 0001 C CNN
 	1    5150 3800
 	1    0    0    -1
@@
 U 1 1 5DAA6A4A
 P 5600 3050
-F 0 "#PWR0131" H 5600 2900 50  0001 C CNN
-F 1 "+3.3V" H 5615 3223 50  0000 C CNN
-F 2 "" H 5600 3050 50  0001 C CNN
-F 3 "" H 5600 3050 50  0001 C CNN
+F 0 "#PWR0131" H 5600 2900 50 0001 C CNN
+F 1 "+3.3V" H 5615 3223 50 0000 C CNN
+F 2 "" H 5600 3050 50 0001 C CNN
+F 3 "" H 5600 3050 50 0001 C CNN
 	1    5600 3050
 	1    0    0    -1
@@
 U 1 1 5DB59EF2
 P 4500 3250
-AR Path="/5DB59EF2" Ref="C?"  Part="1"
-AR Path="/5D7E2E67/5DB59EF2" Ref="C?"  Part="1"
-AR Path="/5D7C5FBE/5DB59EF2" Ref="C?"  Part="1"
-AR Path="/5DAA4BA2/5DB59EF2" Ref="C38"  Part="1"
-F 0 "C38" H 4615 3296 50  0000 L CNN
-F 1 "100n" H 4615 3205 50  0000 L CNN
-F 2 "Capacitor_SMD:C_0603_1608Metric" H 4538 3100 50  0001 C CNN
-F 3 "~" H 4500 3250 50  0001 C CNN
-F 4 "C14663" H 4615 3396 50  0001 C CNN "LCSC Part"
+AR Path="/5DB59EF2" Ref="C?" Part="1"
+AR Path="/5D7E2E67/5DB59EF2" Ref="C?" Part="1"
+AR Path="/5D7C5FBE/5DB59EF2" Ref="C?" Part="1"
+AR Path="/5DAA4BA2/5DB59EF2" Ref="C38" Part="1"
+F 0 "C38" H 4615 3296 50 0000 L CNN
+F 1 "100n" H 4615 3205 50 0000 L CNN
+F 2 "Capacitor_SMD:C_0603_1608Metric" H 4538 3100 50 0001 C CNN
+F 3 "~" H 4500 3250 50 0001 C CNN
+F 4 "0" H 4615 3396 50 0001 C CNN "JLCPCB Rotation"
+F 5 "C14663" H 4615 3396 50 0001 C CNN "LCSC Part"
 	1    4500 3250
 	1    0    0    -1
@@
 U 1 1 5DB59EF8
 P 4500 3050
-AR Path="/5D7C5FBE/5DB59EF8" Ref="#PWR?"  Part="1"
-AR Path="/5DAA4BA2/5DB59EF8" Ref="#PWR0132"  Part="1"
-F 0 "#PWR0132" H 4500 2900 50  0001 C CNN
-F 1 "+3V3" H 4515 3223 50  0000 C CNN
-F 2 "" H 4500 3050 50  0001 C CNN
-F 3 "" H 4500 3050 50  0001 C CNN
+AR Path="/5D7C5FBE/5DB59EF8" Ref="#PWR?" Part="1"
+AR Path="/5DAA4BA2/5DB59EF8" Ref="#PWR0132" Part="1"
+F 0 "#PWR0132" H 4500 2900 50 0001 C CNN
+F 1 "+3V3" H 4515 3223 50 0000 C CNN
+F 2 "" H 4500 3050 50 0001 C CNN
+F 3 "" H 4500 3050 50 0001 C CNN
 	1    4500 3050
 	1    0    0    -1
@@
 U 1 1 5DB59EFE
 P 4500 3450
-AR Path="/5D7C5FBE/5DB59EFE" Ref="#PWR?"  Part="1"
-AR Path="/5DAA4BA2/5DB59EFE" Ref="#PWR0133"  Part="1"
-F 0 "#PWR0133" H 4500 3200 50  0001 C CNN
-F 1 "GND" H 4505 3277 50  0000 C CNN
-F 2 "" H 4500 3450 50  0001 C CNN
-F 3 "" H 4500 3450 50  0001 C CNN
+AR Path="/5D7C5FBE/5DB59EFE" Ref="#PWR?" Part="1"
+AR Path="/5DAA4BA2/5DB59EFE" Ref="#PWR0133" Part="1"
+F 0 "#PWR0133" H 4500 3200 50 0001 C CNN
+F 1 "GND" H 4505 3277 50 0000 C CNN
+F 2 "" H 4500 3450 50 0001 C CNN
+F 3 "" H 4500 3450 50 0001 C CNN
 	1    4500 3450
 	1    0    0    -1

Commit message: Schematic tweaks
Connections:
- net GND: no longer U8.7 (~WC)
- new net ~WC: U8.7 (~WC)
Changed lines of the file:
@@
 encoding utf-8
 Sheet 9 11
-Title ""
+Title "manila iCE"
 Date ""
-Rev ""
+Rev "1.0"
 Comp ""
 Comment1 ""
@@
 Text HLabel 6450 3300 2    50   BiDi ~ 0
 SDA
-Text HLabel 6450 3400 2    50   BiDi ~ 0
+Text HLabel 6450 3400 2    50   Input ~ 0
 SCL
 Text Notes 4600 2300 0    50   ~ 0
@@
 	5600 3050 5600 3100
 Wire Wire Line
-	6000 3500 6050 3500
-Wire Wire Line
-	6050 3500 6050 3750
-Wire Wire Line
-	6050 3750 5600 3750
-Wire Wire Line
 	6000 3400 6450 3400
 Wire Wire Line
@@
 Connection ~ 5150 3500
 Connection ~ 5150 3750
-Connection ~ 5600 3750
+Text HLabel 6450 3500 2    50   Input ~ 0
+~WC
+Wire Wire Line
+	6000 3500 6450 3500
 $EndSCHEMATC
