File: hw/PMOD.sch (KiCad schematic (older format))
At the start: 3 parts, among them J4 Conn_02x06_Odd_Even, U12 SRV05-4, U14 SRV05-4

Commit message: Schematic tweaks
Other:
- note added: "N.B KiCAD pin numbering is different to PMOD spec pin numbering."
- note removed: "N.B Pinout does not match PMOD spec to fit in with KiCAD numbering"
Changed lines of the file:
@@
 $Descr A4 11693 8268
 encoding utf-8
-Sheet 7 11
-Title ""
+Sheet 6 11
+Title "manila iCE"
 Date ""
-Rev ""
+Rev "1.0"
 Comp ""
 Comment1 ""
@@
 AR Path="/5EA5DA36/5EA5FB48" Ref="#PWR0102"  Part="1"
 AR Path="/5EA6C61B/5EA5FB48" Ref="#PWR0106"  Part="1"
-F 0 "#PWR0106" H 6050 3800 50  0001 C CNN
+F 0 "#PWR0102" H 6050 3800 50  0001 C CNN
 F 1 "GND" H 6055 3877 50  0000 C CNN
 F 2 "" H 6050 4050 50  0001 C CNN
@@
 AR Path="/5EA5DA36/5EA6052D" Ref="#PWR0101"  Part="1"
 AR Path="/5EA6C61B/5EA6052D" Ref="#PWR0105"  Part="1"
-F 0 "#PWR0105" H 5450 3800 50  0001 C CNN
+F 0 "#PWR0101" H 5450 3800 50  0001 C CNN
 F 1 "GND" H 5455 3877 50  0000 C CNN
 F 2 "" H 5450 4050 50  0001 C CNN
@@
 AR Path="/5EA5DA36/5EA60E2D" Ref="#PWR0103"  Part="1"
 AR Path="/5EA6C61B/5EA60E2D" Ref="#PWR0107"  Part="1"
-F 0 "#PWR0107" H 6050 3150 50  0001 C CNN
+F 0 "#PWR0103" H 6050 3150 50  0001 C CNN
 F 1 "+3V3" H 6065 3473 50  0000 C CNN
 F 2 "" H 6050 3300 50  0001 C CNN
@@
 AR Path="/5EA5DA36/5EA61156" Ref="#PWR0100"  Part="1"
 AR Path="/5EA6C61B/5EA61156" Ref="#PWR0104"  Part="1"
-F 0 "#PWR0104" H 5450 3150 50  0001 C CNN
+F 0 "#PWR0100" H 5450 3150 50  0001 C CNN
 F 1 "+3V3" H 5465 3473 50  0000 C CNN
 F 2 "" H 5450 3300 50  0001 C CNN
@@
 AR Path="/5EA5DA36/5DB0E5EC" Ref="J4"  Part="1"
 AR Path="/5EA6C61B/5DB0E5EC" Ref="J5"  Part="1"
-F 0 "J5" H 5750 3950 50  0000 C CNN
+F 0 "J4" H 5750 3950 50  0000 C CNN
 F 1 "Conn_02x06_Odd_Even" H 5700 4400 50  0000 C CNN
 F 2 "Connector_PinSocket_2.54mm:PinSocket_2x06_P2.54mm_Horizontal" H 5700 3650 50  0001 C CNN
@@
 AR Path="/5EA5DA36/5DD2B31C" Ref="#PWR0153"  Part="1"
 AR Path="/5EA6C61B/5DD2B31C" Ref="#PWR0155"  Part="1"
-F 0 "#PWR0155" H 4500 6100 50  0001 C CNN
+F 0 "#PWR0153" H 4500 6100 50  0001 C CNN
 F 1 "GND" H 4505 6177 50  0000 C CNN
 F 2 "" H 4500 6350 50  0001 C CNN
@@
 AR Path="/5EA5DA36/5DD2B329" Ref="U12"  Part="1"
 AR Path="/5EA6C61B/5DD2B329" Ref="U13"  Part="1"
-F 0 "U13" H 4250 6250 50  0000 C CNN
+F 0 "U12" H 4250 6250 50  0000 C CNN
 F 1 "SRV05-4" H 4800 6250 50  0000 C CNN
 F 2 "Package_TO_SOT_SMD:SOT-23-6" H 5200 5350 50  0001 C CNN
@@
 AR Path="/5EA5DA36/5DD2F395" Ref="#PWR0152"  Part="1"
 AR Path="/5EA6C61B/5DD2F395" Ref="#PWR0154"  Part="1"
-F 0 "#PWR0154" H 4500 5100 50  0001 C CNN
+F 0 "#PWR0152" H 4500 5100 50  0001 C CNN
 F 1 "+3V3" H 4515 5423 50  0000 C CNN
 F 2 "" H 4500 5250 50  0001 C CNN
@@
 AR Path="/5EA5DA36/5DD3395B" Ref="#PWR0157"  Part="1"
 AR Path="/5EA6C61B/5DD3395B" Ref="#PWR0159"  Part="1"
-F 0 "#PWR0159" H 6250 6100 50  0001 C CNN
+F 0 "#PWR0157" H 6250 6100 50  0001 C CNN
 F 1 "GND" H 6255 6177 50  0000 C CNN
 F 2 "" H 6250 6350 50  0001 C CNN
@@
 AR Path="/5EA5DA36/5DD33963" Ref="U14"  Part="1"
 AR Path="/5EA6C61B/5DD33963" Ref="U15"  Part="1"
-F 0 "U15" H 6000 6250 50  0000 C CNN
+F 0 "U14" H 6000 6250 50  0000 C CNN
 F 1 "SRV05-4" H 6550 6250 50  0000 C CNN
 F 2 "Package_TO_SOT_SMD:SOT-23-6" H 6950 5350 50  0001 C CNN
@@
 AR Path="/5EA5DA36/5DD33971" Ref="#PWR0156"  Part="1"
 AR Path="/5EA6C61B/5DD33971" Ref="#PWR0158"  Part="1"
-F 0 "#PWR0158" H 6250 5100 50  0001 C CNN
+F 0 "#PWR0156" H 6250 5100 50  0001 C CNN
 F 1 "+3V3" H 6265 5423 50  0000 C CNN
 F 2 "" H 6250 5250 50  0001 C CNN
@@
 DATA7
 Text Notes 5050 2150 0    50   ~ 0
-N.B Pinout does not match PMOD spec to fit in with KiCAD numbering
+N.B KiCAD pin numbering is different to PMOD spec pin numbering.
 Text Label 4800 3650 0    50   ~ 0
 DATA6
@@
 Wire Wire Line
 	6250 5250 6250 5300
+Entry Wire Line
+	4650 3550 4750 3650
+Entry Wire Line
+	4650 3650 4750 3750
+Entry Wire Line
+	4650 3750 4750 3850
+Entry Wire Line
+	4650 3850 4750 3950
+Entry Wire Line
+	6900 3550 6800 3650
+Entry Wire Line
+	6900 3650 6800 3750
+Entry Wire Line
+	6900 3750 6800 3850
+Entry Wire Line
+	6900 3850 6800 3950
 Wire Bus Line
 	6900 3350 6900 4400
 Wire Bus Line
 	4650 3300 4650 4400
-Entry Wire Line
-	4650 3550 4750 3650
-Entry Wire Line
-	4650 3650 4750 3750
-Entry Wire Line
-	4650 3750 4750 3850
-Entry Wire Line
-	4650 3850 4750 3950
-Entry Wire Line
-	6900 3550 6800 3650
-Entry Wire Line
-	6900 3650 6800 3750
-Entry Wire Line
-	6900 3750 6800 3850
-Entry Wire Line
-	6900 3850 6800 3950
 $EndSCHEMATC
