File: hw/SDRAM.sch (KiCad schematic (older format))
At the start: 8 parts, among them U1 W9812G6KH-6

Commit message: Fix JLC rotation
Parts:
- C1, C2, C3, C4, C5, C6, C7, U1: JLCPCB Rotation (none) -> 0
